File: source/rtl872xd-dev-board/rtl872xd-dev-board.kicad_pcb (KiCad board)
At the start: 2 copper layers, 0 parts

Commit message: finished prelim layout
Parts:
- added AE1: Antenna_Shield, RF_Antenna_project:AKK_2.4GHz_5GHz_Left, F.Cu at (134.5, 109.0)
- added C1: 0.4p, Capacitor_SMD:C_0402_1005Metric, F.Cu at (136.5, 121.0)
- added C10: 100n, Capacitor_SMD:C_0402_1005Metric, F.Cu at (117.0, 129.0)
- added C11: C, Capacitor_SMD:C_0402_1005Metric, F.Cu at (136.2, 130.8)
- added C12: C, Capacitor_SMD:C_0402_1005Metric, F.Cu at (133.2, 133.8)
- added C13: 1u, Capacitor_SMD:C_0402_1005Metric, F.Cu at (128.8, 134.8)
- added C14: 4.7n, Capacitor_SMD:C_0402_1005Metric, F.Cu at (129.5, 134.0)
- added C15: 2.2u, Capacitor_SMD:C_0402_1005Metric, F.Cu at (124.5, 118.0)
- added C16: 10u, Capacitor_SMD:C_0402_1005Metric, F.Cu at (116.0, 124.5)
- added C17: 100n, Capacitor_SMD:C_0402_1005Metric, F.Cu at (130.2, 133.2)
- added C18: 1n, Capacitor_SMD:C_0402_1005Metric, F.Cu at (133.8, 129.8)
- added C19: 100n, Capacitor_SMD:C_0402_1005Metric, F.Cu at (131.8, 131.8)
- added C2: 0.3p, Capacitor_SMD:C_0402_1005Metric, F.Cu at (135.0, 125.0)
- added C20: 100n, Capacitor_SMD:C_0402_1005Metric, F.Cu at (132.5, 131.0)
- added C21: 100n, Capacitor_SMD:C_0402_1005Metric, F.Cu at (134.5, 129.0)
- added C22: 100n, Capacitor_SMD:C_0402_1005Metric, F.Cu at (135.2, 128.2)
- added C23: 100n, Capacitor_SMD:C_0402_1005Metric, F.Cu at (136.0, 127.5)
- added C24: 100n, Capacitor_SMD:C_0402_1005Metric, F.Cu at (136.8, 126.8)
- added C25: 100n, Capacitor_SMD:C_0402_1005Metric, F.Cu at (133.5, 122.0)
- added C26: 100n, Capacitor_SMD:C_0402_1005Metric, F.Cu at (132.5, 121.0)
- added C27: 100n, Capacitor_SMD:C_0402_1005Metric, F.Cu at (125.2, 117.2)
- added C28: 100n, Capacitor_SMD:C_0402_1005Metric, F.Cu at (122.8, 119.8)
- added C29: 2.2u, Capacitor_SMD:C_0402_1005Metric, F.Cu at (120.2, 122.2)
- added C3: 0.5p, Capacitor_SMD:C_0402_1005Metric, F.Cu at (134.5, 121.0)
- added C30: 100n, Capacitor_SMD:C_0402_1005Metric, F.Cu at (119.5, 123.0)
- added C31: 4.7u, Capacitor_SMD:C_0402_1005Metric, F.Cu at (118.8, 123.8)
- added C32: 100n, Capacitor_SMD:C_0402_1005Metric, F.Cu at (118.0, 124.5)
- added C33: ~, Capacitor_SMD:C_0402_1005Metric, F.Cu at (117.0, 125.5)
- added C34: 2.2u, Capacitor_SMD:C_0402_1005Metric, F.Cu at (118.5, 129.0)
- added C35: 2.2u, Capacitor_SMD:C_0402_1005Metric, F.Cu at (123.8, 133.2)
- added C36: 1u, Capacitor_SMD:C_0402_1005Metric, F.Cu at (128.0, 135.5)
- added C4: 1.0p, Capacitor_SMD:C_0402_1005Metric, F.Cu at (133.5, 123.5)
- added C5: 0R, Capacitor_SMD:C_0402_1005Metric, F.Cu at (135.5, 117.5)
- added C6: 0R, Capacitor_SMD:C_0402_1005Metric, F.Cu at (135.0, 115.5)
- added C7: C, Capacitor_SMD:C_0402_1005Metric, F.Cu at (134.0, 113.0)
- added C8: C, Capacitor_SMD:C_0402_1005Metric, F.Cu at (134.0, 110.0)
- added C9: 1.8p, Capacitor_SMD:C_0402_1005Metric, F.Cu at (136.0, 116.0)
- added DP1: MDPX18M1524P69-D03, RF_Diplexer:DP_0603_1608Metric, F.Cu at (135.5, 119.5)
- added G***: LOGO, LOGO, F.Cu at (119.0, 119.0)
- added J1: Conn_Coaxial, Connector_Coaxial:U.FL_Hirose_U.FL-R-SMT-1_Vertical, F.Cu at (137.5, 112.5)
- added J2: Bus_M.2_Socket_B, Connector_M.2:M.2-B-KEY-22x, F.Cu at (127.0, 145.2)
- added L1: 1n, Inductor_SMD:L_0402_1005Metric, F.Cu at (136.0, 122.5)
- added L2: 3.3n, Inductor_SMD:L_0402_1005Metric, F.Cu at (135.0, 122.5)
- added L3: L, Inductor_SMD:L_0402_1005Metric, F.Cu at (134.5, 111.5)
- added L4: 2.2u, Inductor_SMD:L_0805_2012Metric, F.Cu at (118.8, 127.2)
- added R1: 10k, Resistor_SMD:R_0402_1005Metric, F.Cu at (122.5, 135.0)
- added R2: 10k, Resistor_SMD:R_0402_1005Metric, F.Cu at (131.0, 132.5)
- added R3: 10k, Resistor_SMD:R_0402_1005Metric, F.Cu at (127.2, 136.2)
- added R4: 10k, Resistor_SMD:R_0402_1005Metric, F.Cu at (129.5, 136.2)
- added R5: 12k, Resistor_SMD:R_0402_1005Metric, F.Cu at (124.5, 134.0)
- added R6: 200, Resistor_SMD:R_0402_1005Metric, F.Cu at (121.0, 121.5)
- added R7: 1k, Resistor_SMD:R_0402_1005Metric, F.Cu at (131.0, 134.8)
- added TP1: TestPoint, TestPoint:TestPoint_Pad_D1.0mm, F.Cu at (137.5, 115.0)
- added TP2: TestPoint, TestPoint:TestPoint_Pad_D1.0mm, F.Cu at (134.5, 114.0)
- added U1: RTL8722DM, Package_DFN_QFN_project:QFN-88_EP_10x10_Pitch0.4mm, F.Cu at (127.0, 126.0)
- added U2: W25Q128JVS, Package_SO:SOIC-8_5.23x5.23mm_P1.27mm, F.Cu at (118.0, 134.8)
- added U3: W25Q16JV, Package_USON:USON-8_3.0x2.0mm_P0.5mm, F.Cu at (118.0, 134.8)
- added U4: LM809, Package_TO_SOT_SMD:SOT-23, F.Cu at (132.8, 136.5)
- added Y1: 40MHz, Crystal:Crystal_SMD_2016-4Pin_2.0x1.6mm, F.Cu at (134.8, 132.2)
Routing:
- net +3V3: track 0.00 -> 154.0 mm, vias 0 -> 14
- net VDD: track 0.00 -> 76.4 mm, vias 0 -> 8
- net /PA11: track 0.00 -> 49.4 mm, vias 0 -> 2
- net /PA13: track 0.00 -> 48.3 mm, vias 0 -> 2
- net /PA15: track 0.00 -> 45.8 mm, vias 0 -> 1
- net /PA17: track 0.00 -> 44.3 mm, vias 0 -> 1
- net /PA16: track 0.00 -> 42.7 mm, vias 0 -> 1
- net /PA19: track 0.00 -> 42.5 mm, vias 0 -> 1
- net /PA21: track 0.00 -> 41.0 mm, vias 0 -> 1
- net /PA18: track 0.00 -> 40.8 mm, vias 0 -> 1
- net /PA20: track 0.00 -> 40.2 mm, vias 0 -> 1
- net /PA23: track 0.00 -> 39.1 mm, vias 0 -> 1
- net /PA22: track 0.00 -> 38.0 mm, vias 0 -> 1
- net /PA24: track 0.00 -> 36.4 mm, vias 0 -> 1
- net /PA31: track 0.00 -> 35.3 mm, vias 0 -> 1
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- added copper zone on B.Cu, net GND
- added copper zone on F.Cu, net GND
- added copper zone on In1.Cu, net GND
- added copper zone on In2.Cu, net GND
Other:
- board outline added: 26 x 39.2 mm
- copper layers 2 -> 4
- board text added: "0.0152 mm"
- board text added: "0.0350 mm"
- board text added: "0.2000 mm"
- board text added: "0.2104 mm"
- board text added: "0.8mm JLC7628 Stackup"
- board text added: "7628*1"
- board text added: "Bottom Layer4"
- board text added: "Copper"
- board text added: "Core"
- board text added: "Inner Layer2"
- board text added: "Inner Layer3"
- board text added: "Layer"
- board text added: "Material Type"
- board text added: "Prepreg"
- board text added: "Thickness"
- board text added: "Top Layer1"
