File: source/rtl872xd-dev-board/rtl872xd-dev-board.kicad_sch (KiCad schematic)
At the start: 0 parts

Commit message: finished prelim layout
Parts:
- added J2: Bus_M.2_Socket_B, Connector_M.2:M.2-B-KEY-22x, symbol Connector:Bus_M.2_Socket_B
- added R2: 12k, Resistor_SMD:R_0402_1005Metric, symbol Device:R
- added R2 (x2): 10k, Resistor_SMD:R_0402_1005Metric, symbol Device:R
- added U1: RTL8722DM, Package_DFN_QFN_project:QFN-88_EP_10x10_Pitch0.4mm, symbol MCU_Realtek:RTL8722DM
Connections:
- new net +3V3: J2.2 (3.3V), J2.4 (3.3V), J2.70 (3.3V), J2.72 (3.3V), J2.74 (3.3V), R2.2
- new net GND: J2.11 (GND), J2.27 (GND), J2.3 (GND), J2.33 (GND), J2.39 (GND), J2.45 (GND), J2.5 (GND), J2.51 (GND), J2.57 (GND), J2.71 (GND), J2.73 (GND), R2.1, R2.1
- new net PA0: J2.41 (PERn0/SATA-B+), U1.4 (PA0/MIC_BIAS)
- new net PA1: J2.29 (PERn1/USB3.0-Rx-/SSIC-RxN), U1.7 (PA1/MIC2_N)
- new net PA10: J2.8 (~{W_DISABLE1}), U1.31 (PA10)
- new net PA11: J2.75 (CONFIG_2), U1.32 (PA11)
- new net PA12: J2.6 (~{FULL_CARD_POWER_OFF}), U1.33 (PA12)
- new net PA13: J2.69 (CONFIG_1), U1.34 (PA13)
- new net PA14: J2.1 (CONFIG_3), U1.35 (PA14)
- new net PA15: J2.68 (SUSCLK), U1.36 (PA15)
- new net PA16: J2.54 (~{PEWAKE}), U1.37 (PA16)
- new net PA17: J2.66 (SIM_DETECT), U1.38 (PA17)
- new net PA18: J2.52 (~{CLKREQ}), U1.39 (PA18)
- new net PA19: J2.64 (COEX1), U1.40 (PA19)
- new net PA2: J2.37 (PETp1/USB3.0-Tx+/SSIC-TxP), U1.6 (PA2/MIC2_P)
- new net PA20: J2.50 (~{PERST}), U1.41 (PA20)
- new net PA21: J2.62 (COEX2), U1.42 (PA21)
- new net PA22: J2.48 (GPIO_4), U1.43 (PA22)
- new net PA23: J2.60 (COEX3), U1.44 (PA23)
- new net PA24: J2.44 (GPIO_2), U1.47 (PA24)
- new net PA25: J2.9 (USB_D-), U1.55 (PA25/HSDM)
- new net PA26: J2.7 (USB_D+), U1.54 (PA26/HSDP)
- new net PA27: J2.30 (UIM-RESET), U1.48 (PA27/SWD_DATA)
- new net PA28: J2.40 (GPIO_0), U1.53 (PA28/RREF)
- new net PA30: J2.42 (GPIO_1), U1.51 (PA30/SPS_SEL)
- new net PA31: J2.46 (GPIO_3), U1.49 (PA31)
- new net PA4: J2.35 (PETn1/USB3.0-Tx-/SSIC-TxN), U1.5 (PA4/MIC1_P)
- new net PA5: J2.31 (PERp1/USB3.0-Rx+/SSIC-RxP), U1.8 (PA5/AUXIN_L)
- new net PA6: J2.25 (DPR), U1.9 (PA6/AUXIN_R)
- new net PA7: J2.23 (GPIO_11), U1.12 (PA7/UART_LOG_TXD)
- new net PA8: J2.21 (CONFIG_0), U1.13 (PA8/UART_LOG_RXD)
- new net PA9: J2.10 (GPIO_9/DAS/~{DSS}/~{LED1}), U1.30 (PA9)
- new net PB0: J2.28 (GPIO_8), U1.50 (PB0)
- new net PB1: J2.20 (GPIO_5), U1.57 (PB1/ADC_CH4)
- new net PB18: J2.61 (ANTCTL1), U1.77 (PB18)
- new net PB19: J2.67 (~{RESET}), U1.78 (PB19)
- new net PB2: J2.38 (DEVSLP), U1.56 (PB2/ADC_CH5)
- new net PB20: J2.55 (REFCLKp), U1.79 (PB20)
- new net PB21: J2.63 (ANTCTL2), U1.80 (PB21)
- new net PB22: J2.49 (PETp0/SATA-A+), U1.81 (PB22)
- new net PB23: J2.65 (ANTCTL3), U1.82 (PB23)
- new net PB28: J2.59 (ANTCTL0), R2.2, U1.85 (PB28/AOUTN_R)
- new net PB29: J2.47 (PETn0/SATA-A-), U1.84 (PB29/AOUTP_R)
- new net PB3: J2.36 (UIM-PWR), U1.58 (PB3/ADC_CH6/SWD_CLK)
- new net PB30: J2.53 (REFCLKn), R2.1, R2.2, U1.86 (PB30/AOUTN_L)
- new net PB31: J2.43 (PERp0/SATA-B-), U1.87 (PB31/AOUTP_L)
- new net PB4: J2.22 (GPIO_6), U1.59 (PB4/TOUCH_KEY0)
- new net PB5: J2.34 (UIM-DATA), U1.60 (PB5/TOUCH_KEY1)
- new net PB6: J2.24 (GPIO_7), U1.61 (PB6/TOUCH_KEY2)
- new net PB7: J2.32 (UIM-CLK), U1.62 (PB7/TOUCH_KEY3)
- new net VBAT_MEAS: J2.26 (GPIO_10)
Other:
- added sheet Flash (Flash.kicad_sch)
- added sheet Power & Clock (Power_Clock.kicad_sch)
- added sheet RF (RF.kicad_sch)
- note added: "48 I/O"
- note added: "PU:SPS PD:LDO"
