File: source/rtl872xd-dev-board/Flash.kicad_sch (KiCad schematic)
At the start: 5 parts, among them U1 RTL8722DM, U3 W25Q128JVS, U6 W25Q16JV

Commit message: resolve all ERC error, reduce number of warnings
Connections:
- net +3V3 renamed +3.3V
Changed lines of the file:
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@@
       (effects (font (size 1.27 1.27)) hide)
     )
-    (property "Datasheet" "https://datasheet.lcsc.com/lcsc/2205311900_UNI-ROYAL-Uniroyal-Elec-0402WGF100KTCE_C25086.pdf" (at 116.84 55.88 0)
+    (property "Datasheet" "~" (at 116.84 55.88 0)
       (effects (font (size 1.27 1.27)) hide)
     )
@@
     )
   )
-  (symbol (lib_id "power:+3V3") (at 124.46 54.61 0) (unit 1)
-    (in_bom yes) (on_board yes) (dnp no) (fields_autoplaced)
-    (property "Reference" "#PWR092" (at 124.46 58.42 0)
-      (effects (font (size 1.27 1.27)) hide)
-    )
-    (property "Value" "+3V3" (at 124.46 49.53 0)
+  (symbol (lib_id "power:GND") (at 124.46 130.81 0) (unit 1)
+    (in_bom yes) (on_board yes) (dnp no) (fields_autoplaced)
+    (property "Reference" "#PWR0105" (at 124.46 137.16 0)
+      (effects (font (size 1.27 1.27)) hide)
+    )
+    (property "Value" "GND" (at 124.46 135.89 0)
+      (effects (font (size 1.27 1.27)))
+    )
+    (property "Footprint" "" (at 124.46 130.81 0)
+      (effects (font (size 1.27 1.27)) hide)
+    )
+    (property "Datasheet" "" (at 124.46 130.81 0)
+      (effects (font (size 1.27 1.27)) hide)
+    )
+    (pin "1")
+    (instances
+      (project "chubby-hat"
+        (path "/4807f255-cede-4a86-b009-c3f93cadbbb8/e072f2d0-1d9f-486d-9f7d-b187c6021c47"
+          (reference "#PWR0105") (unit 1)
+        )
+      )
+      (project "rtl872xd-dev-board"
+        (path "/5477044b-5ae5-4ed6-bb7d-f5f3cc95a2d4"
+          (reference "#PWR017") (unit 1)
+        )
+        (path "/5477044b-5ae5-4ed6-bb7d-f5f3cc95a2d4/88b15939-7f22-492e-8320-edd70a2f1bdd"
+          (reference "#PWR016") (unit 1)
+        )
+      )
+    )
+  )
+  (symbol (lib_id "power:+3.3V") (at 124.46 54.61 0) (unit 1)
+    (in_bom yes) (on_board yes) (dnp no) (fields_autoplaced)
+    (property "Reference" "#PWR013" (at 124.46 58.42 0)
+      (effects (font (size 1.27 1.27)) hide)
+    )
+    (property "Value" "+3.3V" (at 124.46 50.8 0)
       (effects (font (size 1.27 1.27)))
     )
@@
     (pin "1")
     (instances
-      (project "chubby-hat"
-        (path "/4807f255-cede-4a86-b009-c3f93cadbbb8/e072f2d0-1d9f-486d-9f7d-b187c6021c47"
-          (reference "#PWR092") (unit 1)
-        )
-      )
-      (project "rtl872xd-dev-board"
-        (path "/5477044b-5ae5-4ed6-bb7d-f5f3cc95a2d4"
-          (reference "#PWR014") (unit 1)
-        )
+      (project "rtl872xd-dev-board"
         (path "/5477044b-5ae5-4ed6-bb7d-f5f3cc95a2d4/88b15939-7f22-492e-8320-edd70a2f1bdd"
           (reference "#PWR013") (unit 1)
-        )
-      )
-    )
-  )
-  (symbol (lib_id "power:GND") (at 124.46 130.81 0) (unit 1)
-    (in_bom yes) (on_board yes) (dnp no) (fields_autoplaced)
-    (property "Reference" "#PWR0105" (at 124.46 137.16 0)
-      (effects (font (size 1.27 1.27)) hide)
-    )
-    (property "Value" "GND" (at 124.46 135.89 0)
-      (effects (font (size 1.27 1.27)))
-    )
-    (property "Footprint" "" (at 124.46 130.81 0)
-      (effects (font (size 1.27 1.27)) hide)
-    )
-    (property "Datasheet" "" (at 124.46 130.81 0)
-      (effects (font (size 1.27 1.27)) hide)
-    )
-    (pin "1")
-    (instances
-      (project "chubby-hat"
-        (path "/4807f255-cede-4a86-b009-c3f93cadbbb8/e072f2d0-1d9f-486d-9f7d-b187c6021c47"
-          (reference "#PWR0105") (unit 1)
-        )
-      )
-      (project "rtl872xd-dev-board"
-        (path "/5477044b-5ae5-4ed6-bb7d-f5f3cc95a2d4"
-          (reference "#PWR017") (unit 1)
-        )
-        (path "/5477044b-5ae5-4ed6-bb7d-f5f3cc95a2d4/88b15939-7f22-492e-8320-edd70a2f1bdd"
-          (reference "#PWR016") (unit 1)
         )
       )
@@
     )
   )
+  (symbol (lib_id "power:+3.3V") (at 124.46 102.87 0) (unit 1)
+    (in_bom yes) (on_board yes) (dnp no) (fields_autoplaced)
+    (property "Reference" "#PWR015" (at 124.46 106.68 0)
+      (effects (font (size 1.27 1.27)) hide)
+    )
+    (property "Value" "+3.3V" (at 124.46 99.06 0)
+      (effects (font (size 1.27 1.27)))
+    )
+    (property "Footprint" "" (at 124.46 102.87 0)
+      (effects (font (size 1.27 1.27)) hide)
+    )
+    (property "Datasheet" "" (at 124.46 102.87 0)
+      (effects (font (size 1.27 1.27)) hide)
+    )
+    (pin "1")
+    (instances
+      (project "rtl872xd-dev-board"
+        (path "/5477044b-5ae5-4ed6-bb7d-f5f3cc95a2d4/88b15939-7f22-492e-8320-edd70a2f1bdd"
+          (reference "#PWR015") (unit 1)
+        )
+      )
+    )
+  )
   (symbol (lib_id "power:GND") (at 134.62 57.15 0) (unit 1)
     (in_bom yes) (on_board yes) (dnp no) (fields_autoplaced)
@@
         )
       )
-    )
-  )
-  (symbol (lib_id "power:+3V3") (at 124.46 102.87 0) (unit 1)
-    (in_bom yes) (on_board yes) (dnp no) (fields_autoplaced)
-    (property "Reference" "#PWR0104" (at 124.46 106.68 0)
-      (effects (font (size 1.27 1.27)) hide)
-    )
-    (property "Value" "+3V3" (at 124.46 97.79 0)
-      (effects (font (size 1.27 1.27)))
-    )
-    (property "Footprint" "" (at 124.46 102.87 0)
-      (effects (font (size 1.27 1.27)) hide)
-    )
-    (property "Datasheet" "" (at 124.46 102.87 0)
-      (effects (font (size 1.27 1.27)) hide)
-    )
-    (pin "1")
-    (instances
-      (project "chubby-hat"
-        (path "/4807f255-cede-4a86-b009-c3f93cadbbb8/e072f2d0-1d9f-486d-9f7d-b187c6021c47"
-          (reference "#PWR0104") (unit 1)
-        )
-      )
-      (project "rtl872xd-dev-board"
-        (path "/5477044b-5ae5-4ed6-bb7d-f5f3cc95a2d4"
-          (reference "#PWR016") (unit 1)
-        )
-        (path "/5477044b-5ae5-4ed6-bb7d-f5f3cc95a2d4/88b15939-7f22-492e-8320-edd70a2f1bdd"
-          (reference "#PWR015") (unit 1)
-        )
-      )

Commit message: tidied up like Marie Kondo
Parts:
- R14: now left out of the parts list
Other:
- moved on the sheet: C10, R14, U1D, U3, U6

Commit message: first production version
Parts:
- U1: now left out of the parts list
Changed lines of the file:
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@@
   )
   (symbol (lib_id "MCU_Realtek:RTL8722DM") (at 27.94 40.64 0) (unit 4)
-    (in_bom yes) (on_board yes) (dnp no) (fields_autoplaced)
+    (in_bom no) (on_board yes) (dnp no) (fields_autoplaced)
     (property "Reference" "U1" (at 27.94 26.67 0)
       (effects (font (size 1.27 1.27)))
