File: source/rtl872xd-dev-board/Power_Clock.kicad_sch (KiCad schematic)
At the start: 33 parts, among them U1 RTL8722DM, U4 LM809, Y1 40MHz

Commit message: resolve all ERC error, reduce number of warnings
Connections:
- net +3V3 renamed +3.3V
Other:
- moved on the sheet: R6

Commit message: tidied up like Marie Kondo
Parts:
- C10, C11, C12: now left out of the parts list
Changed lines of the file:
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@@
   )
   (symbol (lib_id "Device:C") (at 68.58 139.7 0) (unit 1)
-    (in_bom yes) (on_board yes) (dnp yes)
+    (in_bom no) (on_board yes) (dnp yes)
     (property "Reference" "C12" (at 71.501 138.5316 0)
       (effects (font (size 1.27 1.27)) (justify left))
@@
   )
   (symbol (lib_id "Device:C") (at 58.42 139.7 0) (unit 1)
-    (in_bom yes) (on_board yes) (dnp yes)
+    (in_bom no) (on_board yes) (dnp yes)
     (property "Reference" "C11" (at 55.499 138.5316 0)
       (effects (font (size 1.27 1.27)) (justify right))
@@
   )
   (symbol (lib_id "Device:C") (at 162.56 114.3 180) (unit 1)
-    (in_bom yes) (on_board yes) (dnp yes) (fields_autoplaced)
+    (in_bom no) (on_board yes) (dnp yes) (fields_autoplaced)
     (property "Reference" "C10" (at 166.37 114.935 0)
       (effects (font (size 1.27 1.27)) (justify right))

Commit message: first production version
Parts:
- added TP3 (x4): TestPoint, TestPoint:TestPoint_Pad_D1.0mm, symbol Connector:TestPoint
- C10: value ~ -> C
- U1: now left out of the parts list
Connections:
- net +3.3V: now also TP3.1
- net CHIP_EN: now also TP3.1
- net GND: now also TP3.1
- net VDD: now also TP3.1
Changed lines of the file:
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@@
   (junction (at 119.38 78.74) (diameter 0) (color 0 0 0 0)
   )
+  (junction (at 50.8 119.38) (diameter 0) (color 0 0 0 0)
+  )
   (junction (at 83.82 50.8) (diameter 0) (color 0 0 0 0)
   )
@@
   (junction (at 43.18 88.9) (diameter 0) (color 0 0 0 0)
   )
+  (junction (at 101.6 134.62) (diameter 0) (color 0 0 0 0)
+  )
   (junction (at 162.56 78.74) (diameter 0) (color 0 0 0 0)
   )
@@
     (stroke (width 0) (type default))
   )
+  (wire (pts (xy 100.33 134.62) (xy 101.6 134.62))
+    (stroke (width 0) (type default))
+  )
   (wire (pts (xy 134.62 116.84) (xy 147.32 116.84))
     (stroke (width 0) (type default))
@@
     (stroke (width 0) (type default))
   )
+  (wire (pts (xy 83.82 49.53) (xy 83.82 50.8))
+    (stroke (width 0) (type default))
+  )
   (wire (pts (xy 68.58 127) (xy 68.58 134.62))
     (stroke (width 0) (type default))
@@
     (stroke (width 0) (type default))
   )
+  (wire (pts (xy 49.53 119.38) (xy 50.8 119.38))
+    (stroke (width 0) (type default))
+  )
   (wire (pts (xy 101.6 134.62) (xy 104.14 134.62))
     (stroke (width 0) (type default))
@@
     (stroke (width 0) (type default))
   )
+  (wire (pts (xy 111.76 36.83) (xy 111.76 38.1))
+    (stroke (width 0) (type default))
+  )
   (wire (pts (xy 99.06 38.1) (xy 101.6 38.1))
     (stroke (width 0) (type default))
@@
     (stroke (width 0) (type default))
   )
+  (wire (pts (xy 50.8 119.38) (xy 50.8 114.3))
+    (stroke (width 0) (type default))
+  )
   (wire (pts (xy 114.3 38.1) (xy 114.3 73.66))
     (stroke (width 0) (type default))
@@
     (stroke (width 0) (type default))
   )
-  (wire (pts (xy 50.8 127) (xy 50.8 114.3))
+  (wire (pts (xy 50.8 127) (xy 50.8 119.38))
     (stroke (width 0) (type default))
   )
@@
     )
   )
+  (symbol (lib_id "Connector:TestPoint") (at 49.53 119.38 90) (unit 1)
+    (in_bom yes) (on_board yes) (dnp no) (fields_autoplaced)
+    (property "Reference" "TP3" (at 46.228 114.3 90)
+      (effects (font (size 1.27 1.27)))
+    )
+    (property "Value" "TestPoint" (at 46.228 116.84 90)
+      (effects (font (size 1.27 1.27)))
+    )
+    (property "Footprint" "TestPoint:TestPoint_Pad_D1.0mm" (at 49.53 114.3 0)
+      (effects (font (size 1.27 1.27)) hide)
+    )
+    (property "Datasheet" "~" (at 49.53 114.3 0)
+      (effects (font (size 1.27 1.27)) hide)
+    )
+    (pin "1")
+    (instances
+      (project "rtl872xd-dev-board"
+        (path "/5477044b-5ae5-4ed6-bb7d-f5f3cc95a2d4/bdc7329f-2717-4429-9357-eafb26421b20"
+          (reference "TP3") (unit 1)
+        )
+        (path "/5477044b-5ae5-4ed6-bb7d-f5f3cc95a2d4/05d3bf15-498f-4c9e-a533-1ff4c5c2cb4b"
+          (reference "TP5") (unit 1)
+        )
+      )
+    )
+  )
   (symbol (lib_id "power:GND") (at 63.5 130.81 180) (unit 1)
     (in_bom yes) (on_board yes) (dnp no)
@@
       (effects (font (size 1.27 1.27)) (justify right))
     )
-    (property "Value" "~" (at 166.37 116.205 0)
+    (property "Value" "C" (at 166.37 116.205 0)
       (effects (font (size 1.27 1.27)) (justify right))
     )
@@
         (path "/5477044b-5ae5-4ed6-bb7d-f5f3cc95a2d4/05d3bf15-498f-4c9e-a533-1ff4c5c2cb4b"
           (reference "C33") (unit 1)
+        )
+      )
+    )
+  )
+  (symbol (lib_id "Connector:TestPoint") (at 100.33 134.62 90) (unit 1)
+    (in_bom yes) (on_board yes) (dnp no) (fields_autoplaced)
+    (property "Reference" "TP3" (at 97.028 129.54 90)
+      (effects (font (size 1.27 1.27)))
+    )
+    (property "Value" "TestPoint" (at 97.028 132.08 90)
+      (effects (font (size 1.27 1.27)))
+    )
+    (property "Footprint" "TestPoint:TestPoint_Pad_D1.0mm" (at 100.33 129.54 0)
+      (effects (font (size 1.27 1.27)) hide)
+    )
+    (property "Datasheet" "~" (at 100.33 129.54 0)
+      (effects (font (size 1.27 1.27)) hide)
+    )
+    (pin "1")
+    (instances
+      (project "rtl872xd-dev-board"
+        (path "/5477044b-5ae5-4ed6-bb7d-f5f3cc95a2d4/bdc7329f-2717-4429-9357-eafb26421b20"
+          (reference "TP3") (unit 1)
+        )
+        (path "/5477044b-5ae5-4ed6-bb7d-f5f3cc95a2d4/05d3bf15-498f-4c9e-a533-1ff4c5c2cb4b"
+          (reference "TP8") (unit 1)
         )
       )
@@
     )
   )
+  (symbol (lib_id "Connector:TestPoint") (at 83.82 49.53 0) (unit 1)
+    (in_bom yes) (on_board yes) (dnp no) (fields_autoplaced)
+    (property "Reference" "TP3" (at 86.36 45.593 0)
+      (effects (font (size 1.27 1.27)) (justify left))
+    )
+    (property "Value" "TestPoint" (at 86.36 48.133 0)
+      (effects (font (size 1.27 1.27)) (justify left))
+    )
+    (property "Footprint" "TestPoint:TestPoint_Pad_D1.0mm" (at 88.9 49.53 0)
+      (effects (font (size 1.27 1.27)) hide)
+    )
+    (property "Datasheet" "~" (at 88.9 49.53 0)
+      (effects (font (size 1.27 1.27)) hide)
+    )
+    (pin "1")
+    (instances
+      (project "rtl872xd-dev-board"
+        (path "/5477044b-5ae5-4ed6-bb7d-f5f3cc95a2d4/bdc7329f-2717-4429-9357-eafb26421b20"
+          (reference "TP3") (unit 1)
+        )
+        (path "/5477044b-5ae5-4ed6-bb7d-f5f3cc95a2d4/05d3bf15-498f-4c9e-a533-1ff4c5c2cb4b"
+          (reference "TP6") (unit 1)
+        )
+      )
+    )
+  )
   (symbol (lib_id "power:GND") (at 157.48 129.54 0) (unit 1)
     (in_bom yes) (on_board yes) (dnp no) (fields_autoplaced)
@@
         (path "/5477044b-5ae5-4ed6-bb7d-f5f3cc95a2d4/05d3bf15-498f-4c9e-a533-1ff4c5c2cb4b"
           (reference "#PWR019") (unit 1)
+        )
+      )
+    )
+  )
+  (symbol (lib_id "Connector:TestPoint") (at 111.76 36.83 0) (unit 1)
+    (in_bom yes) (on_board yes) (dnp no) (fields_autoplaced)
+    (property "Reference" "TP3" (at 114.3 32.893 0)
+      (effects (font (size 1.27 1.27)) (justify left))
+    )
+    (property "Value" "TestPoint" (at 114.3 35.433 0)
+      (effects (font (size 1.27 1.27)) (justify left))
+    )
+    (property "Footprint" "TestPoint:TestPoint_Pad_D1.0mm" (at 116.84 36.83 0)
+      (effects (font (size 1.27 1.27)) hide)
+    )
+    (property "Datasheet" "~" (at 116.84 36.83 0)
+      (effects (font (size 1.27 1.27)) hide)
+    )
+    (pin "1")
+    (instances
+      (project "rtl872xd-dev-board"
+        (path "/5477044b-5ae5-4ed6-bb7d-f5f3cc95a2d4/bdc7329f-2717-4429-9357-eafb26421b20"
+          (reference "TP3") (unit 1)
+        )
+        (path "/5477044b-5ae5-4ed6-bb7d-f5f3cc95a2d4/05d3bf15-498f-4c9e-a533-1ff4c5c2cb4b"
+          (reference "TP7") (unit 1)
         )
       )
@@
   )
   (symbol (lib_id "MCU_Realtek:RTL8722DM") (at 104.14 114.3 0) (unit 1)
-    (in_bom yes) (on_board yes) (dnp no) (fields_autoplaced)
+    (in_bom no) (on_board yes) (dnp no) (fields_autoplaced)
     (property "Reference" "U1" (at 108.6359 132.08 0)
       (effects (font (size 1.27 1.27)) (justify left))
