File: source/rtl872xd-dev-board/RF.kicad_sch (KiCad schematic)
At the start: 18 parts, among them J1 Conn_Coaxial, U1 RTL8722DM

Commit message: tidied up like Marie Kondo
Parts:
- C9: now left out of the parts list
Other:
- moved on the sheet: AE2, C1, C2, C3, C4, C5, C6, C7, C8, C9, DP1, J1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

Commit message: first production version
Parts:
- C1: LCSC (none) -> C387964; MPN (none) -> V0R3B0402C0G500NBT
- C2: LCSC (none) -> C610035; MPN (none) -> 0603N0R3C500CT
- C3: LCSC (none) -> C152789; MPN (none) -> 0402N0R5C500CT
- C7, C8: now not fitted; now left out of the parts list
- J1: LCSC (none) -> C4749207; MPN (none) -> IPEX-SMD
- L1: LCSC (none) -> C74299; MPN (none) -> SDCL1005C1N0STDFM01
- L2: LCSC (none) -> C280259; MPN (none) -> CS0402-3N3H-S
- L3: value L -> 1n(0.9n); LCSC (none) -> C74299; MPN (none) -> SDCL1005C1N0STDFM01
- TP1, TP2: LCSC n/a -> (none); MPN n/a -> (none)
- U1: now left out of the parts list
Changed lines of the file:
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@@
       (effects (font (size 1.27 1.27)) hide)
     )
-    (property "LCSC" "n/a" (at 119.38 24.13 0)
-      (effects (font (size 1.27 1.27)) hide)
-    )
-    (property "MPN" "n/a" (at 119.38 24.13 0)
+    (property "LCSC" "" (at 119.38 24.13 0)
+      (effects (font (size 1.27 1.27)) hide)
+    )
+    (property "MPN" "" (at 119.38 24.13 0)
       (effects (font (size 1.27 1.27)) hide)
     )
@@
       (effects (font (size 1.27 1.27)) hide)
     )
+    (property "LCSC" "C610035" (at 66.04 38.1 0)
+      (effects (font (size 1.27 1.27)) hide)
+    )
+    (property "MPN" "0603N0R3C500CT" (at 66.04 38.1 0)
+      (effects (font (size 1.27 1.27)) hide)
+    )
     (pin "1")
     (pin "2")
@@
   )
   (symbol (lib_id "Device:C") (at 162.56 50.8 0) (unit 1)
-    (in_bom yes) (on_board yes) (dnp no) (fields_autoplaced)
+    (in_bom no) (on_board yes) (dnp yes) (fields_autoplaced)
     (property "Reference" "C8" (at 166.37 50.165 0)
       (effects (font (size 1.27 1.27)) (justify left))
@@
     )
     (property "Datasheet" "~" (at 71.12 58.42 0)
+      (effects (font (size 1.27 1.27)) hide)
+    )
+    (property "LCSC" "C280259" (at 71.12 58.42 0)
+      (effects (font (size 1.27 1.27)) hide)
+    )
+    (property "MPN" "CS0402-3N3H-S" (at 71.12 58.42 0)
       (effects (font (size 1.27 1.27)) hide)
     )
@@
   )
   (symbol (lib_id "Device:C") (at 152.4 50.8 0) (unit 1)
-    (in_bom yes) (on_board yes) (dnp no) (fields_autoplaced)
+    (in_bom no) (on_board yes) (dnp yes) (fields_autoplaced)
     (property "Reference" "C7" (at 156.21 50.165 0)
       (effects (font (size 1.27 1.27)) (justify left))
@@
       (effects (font (size 1.27 1.27)))
     )
-    (property "Value" "L" (at 157.48 44.45 90)
+    (property "Value" "1n(0.9n)" (at 157.48 44.45 90)
       (effects (font (size 1.27 1.27)))
     )
@@
       (effects (font (size 1.27 1.27)) hide)
     )
+    (property "LCSC" "C74299" (at 157.48 45.72 0)
+      (effects (font (size 1.27 1.27)) hide)
+    )
+    (property "MPN" "SDCL1005C1N0STDFM01" (at 157.48 45.72 0)
+      (effects (font (size 1.27 1.27)) hide)
+    )
     (pin "1")
     (pin "2")
@@
       (effects (font (size 1.27 1.27)) hide)
     )
+    (property "LCSC" "C152789" (at 76.2 63.5 0)
+      (effects (font (size 1.27 1.27)) hide)
+    )
+    (property "MPN" "0402N0R5C500CT" (at 76.2 63.5 0)
+      (effects (font (size 1.27 1.27)) hide)
+    )
     (pin "1")
     (pin "2")
@@
       (effects (font (size 1.27 1.27)) hide)
     )
+    (property "LCSC" "C4749207" (at 127 25.4 0)
+      (effects (font (size 1.27 1.27)) hide)
+    )
+    (property "MPN" "IPEX-SMD" (at 127 25.4 0)
+      (effects (font (size 1.27 1.27)) hide)
+    )
     (pin "1")
     (pin "2")
@@
       (effects (font (size 1.27 1.27)) hide)
     )
+    (property "LCSC" "C387964" (at 76.2 38.1 0)
+      (effects (font (size 1.27 1.27)) hide)
+    )
+    (property "MPN" "V0R3B0402C0G500NBT" (at 76.2 38.1 0)
+      (effects (font (size 1.27 1.27)) hide)
+    )
     (pin "1")
     (pin "2")
@@
       (effects (font (size 1.27 1.27)) hide)
     )
+    (property "LCSC" "C74299" (at 71.12 33.02 0)
+      (effects (font (size 1.27 1.27)) hide)
+    )
+    (property "MPN" "SDCL1005C1N0STDFM01" (at 71.12 33.02 0)
+      (effects (font (size 1.27 1.27)) hide)
+    )
     (pin "1")
     (pin "2")
@@
   )
   (symbol (lib_id "MCU_Realtek:RTL8722DM") (at 33.02 50.8 0) (unit 3)
-    (in_bom yes) (on_board yes) (dnp no) (fields_autoplaced)
+    (in_bom no) (on_board yes) (dnp no) (fields_autoplaced)
     (property "Reference" "U1" (at 33.02 34.29 0)
       (effects (font (size 1.27 1.27)))
@@
       (effects (font (size 1.27 1.27)) hide)
     )
-    (property "LCSC" "n/a" (at 137.16 44.45 0)
-      (effects (font (size 1.27 1.27)) hide)
-    )
-    (property "MPN" "n/a" (at 137.16 44.45 0)
-      (effects (font (size 1.27 1.27)) hide)
-    )
+    (property "LCSC" "" (at 137.16 44.45 0)
+      (effects (font (size 1.27 1.27)) hide)
+    )
+    (property "MPN" "" (at 137.16 44.45 0)
+      (effects (font (size 1.27 1.27)) hide)
+    )
